File: eagle/CR78-MB.sch (EAGLE design)
At the start: 45 parts, among them Q508 2N3904, Q518 2N3904, Q519 2N3904, Q520 2N3904, Q521 2N3904, Q7 2N3904

Commit message: half schemo
Parts:
- removed 671, R543: 82k, rcl:R-US_0207/7
- removed C4, C5: 68n, rcl:C-US050-025X075
- removed C507: 100/10, rcl:CPOL-USB45181A
- removed C531: 22n, rcl:C-US050-025X075
- removed D519, D520, D527: (no value), SparkFun-DiscreteSemi:DIODE1N4148
- removed GU: (no value), con-molex:22-23-2061
- removed Q519, Q520, Q521: 2N3904, 808_lt:2N3904
- removed R544, R545: 56k, rcl:R-US_0207/7
- removed R546: 2M2, rcl:R-US_0207/7
- removed R549, R670, R675: 10k, rcl:R-US_0207/7
- removed R550: 820, rcl:R-US_0207/7
- removed R672: 47k, rcl:R-US_0207/7
- removed R673: 5k6, rcl:R-US_0207/7
- removed R674: 15k, rcl:R-US_0207/7
- removed R676: 3k9, rcl:R-US_0207/7
- removed R677: 18k, rcl:R-US_0207/7
- removed VR59: 100K, TR808clone:TRIM_EU-B64Y
- added C540: 22n, rcl:C-US050-025X075
- added C541: 15n, rcl:C-US050-025X075
- added D524: (no value), SparkFun-DiscreteSemi:DIODE1N4148
- added IC1: 40106N, 40xx:40106N
- added MB: 22-23-2051, con-molex:22-23-2051
- added Q1: 2N3904, 808_lt:2N3904
- added R566: 470k, rcl:R-US_0207/7
- added R567: 820k, rcl:R-US_0207/7
- added R568: 10k, rcl:R-US_0207/7
- added R569: 4M7, rcl:R-US_0207/7
- C342: value 15n -> 18n
- R548: value 470k -> 270k
- R570: value 47k -> 100k
- R668: value 56k -> 10k
- renumbered C532 to C342, Q508 to Q510, R547 to R570
Connections:
- removed net N$10: R673.1, R674.1, R675.1, R676.2
- removed net N$11: GU-2.S, R668.1
- removed net N$14: R545.1, VR59.A
- removed net N$22: R543.1, R544.1, R545.2, R672.2
- removed net N$23: D527.C, R672.1
- removed net N$46: D527.A, Q519.C, R670.2
- removed net N$47: Q519.B, R668.2
- removed net N$5: D520.C, Q521.C, R546.2, R675.2
- removed net N$6: C5.2, D520.A, R674.2
- removed net N$8: C4.2, Q521.B, R544.2
- removed net N$9: C4.1, Q520.C, R673.2
- new net +5V: MB-2.S
- net +12V: now also MB-3.S, R567.2, R568.2, R668.2; no longer GU-4.S, R549.1, R670.1, R676.1, VR59.E, VR59.S
- net GND: now also C540.2, MB-4.S, Q1.E, Q510.E, R548.1; no longer C507.-, GU-5.S, Q519.E, R550.2, R677.1
- net N$1: now also D524.A, Q1.C, R568.1; no longer 671.2, D519.C, R677.2
- net N$12: now also C541.1, R569.2; no longer C531.1, R546.1
- net N$17: now also C541.2; no longer C531.2
- net N$2: now also Q1.B, R566.1, R567.1; no longer C5.1, D519.A, Q520.B, R543.2
- net N$20: now also R566.2; no longer 671.1
- net N$24: now also MB-1.S; no longer GU-1.S
- net N$27: now also R668.1
- net N$3: no longer GU-3.S
- net N$4: now also C540.1, D524.C, R569.1; no longer C507.+, Q510.E, Q520.E, Q521.E, R548.1, R549.2, R550.1
- net N$7: now also MB-5.S; no longer GU-6.S
Other:
- note removed: "NOISE"
- moved on the sheet: C1, C2, C3, JCK1, Q518, Q7, R1, R2, R3, R4, R667, R668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

Commit message: schemo
Parts:
- removed VR63: 50KB, TR808clone:TRIM_EU-B64Y
- added C4: 1n5, rcl:C-US050-025X075
- added C5: 1n8, rcl:C-US050-025X075
- added C6: 2n2, rcl:C-US050-025X075
- added R10, R5, R9: 4k7, rcl:R-US_0207/7
- added R11, R12, R7: 470k, rcl:R-US_0207/7
- added R13, R6, R8: 39k, rcl:R-US_0207/7
- added R14: 10k, rcl:R-US_0207/7
- added VR1, VR2, VR3: 20K, TR808clone:TRIM_EU-B64Y
Connections:
- new net N$10: IC1E.O, IC1F.I, R13.1
- new net N$11: C5.2, IC1D.O, R11.2
- new net N$14: C6.2, IC1F.O, R12.2
- new net N$22: C4.2, IC1B.O, R7.2
- new net N$23: R6.2, VR1.E
- new net N$25: R8.2, VR2.E
- new net N$26: R13.2, VR3.E
- new net N$28: C4.1, R5.2, VR1.S
- new net N$29: C5.1, R9.2, VR2.S
- new net N$30: C6.1, R10.2, VR3.S
- new net N$5: IC1A.O, IC1B.I, R6.1
- new net N$6: IC1C.O, IC1D.I, R8.1
- new net N$8: IC1C.I, R9.1
- new net N$9: IC1E.I, R10.1
- net +12V: no longer VR63.A
- net +5V: now also IC1P.VDD
- net GND: now also IC1P.VSS, R14.2
- net N$17: now also IC1A.I, R5.1; no longer C541.2, VR63.S
- net N$3: now also C541.2, R11.1, R12.1, R14.1, R7.1; no longer VR63.E
Other:
- moved on the sheet: C2, IC1A, R1, R2, R3, R4

Commit message: starting brd
Parts:
- renumbered D524 to D571, L4 to L6, Q1 to Q526
Other:
- moved on the sheet: C4, C5, C6, IC1C, IC1D, IC1E, IC1F, R10, R11, R12, R13, R8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

Commit message: parts on the brd
Parts:
- C2: device rcl:C-US050-025X075 -> rcl:C-US025-030X050
Changed lines of the file:
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@@
 <grid distance="0.1" unitdist="inch" unit="inch" style="lines" multiple="1" display="no" altdistance="0.01" altunitdist="inch" altunit="inch"/>
 <layers>
-<layer number="1" name="Top" color="4" fill="1" visible="no" active="no"/>
-<layer number="16" name="Bottom" color="1" fill="1" visible="no" active="no"/>
-<layer number="17" name="Pads" color="2" fill="1" visible="no" active="no"/>
-<layer number="18" name="Vias" color="2" fill="1" visible="no" active="no"/>
-<layer number="19" name="Unrouted" color="6" fill="1" visible="no" active="no"/>
-<layer number="20" name="Dimension" color="15" fill="1" visible="no" active="no"/>
-<layer number="21" name="tPlace" color="7" fill="1" visible="no" active="no"/>
-<layer number="22" name="bPlace" color="7" fill="1" visible="no" active="no"/>
-<layer number="23" name="tOrigins" color="15" fill="1" visible="no" active="no"/>
-<layer number="24" name="bOrigins" color="15" fill="1" visible="no" active="no"/>
-<layer number="25" name="tNames" color="7" fill="1" visible="no" active="no"/>
-<layer number="26" name="bNames" color="7" fill="1" visible="no" active="no"/>
-<layer number="27" name="tValues" color="7" fill="1" visible="no" active="no"/>
-<layer number="28" name="bValues" color="7" fill="1" visible="no" active="no"/>
+<layer number="1" name="Top" color="4" fill="1" visible="yes" active="no"/>
+<layer number="16" name="Bottom" color="1" fill="1" visible="yes" active="no"/>
+<layer number="17" name="Pads" color="2" fill="1" visible="yes" active="no"/>
+<layer number="18" name="Vias" color="2" fill="1" visible="yes" active="no"/>
+<layer number="19" name="Unrouted" color="6" fill="1" visible="yes" active="no"/>
+<layer number="20" name="Dimension" color="15" fill="1" visible="yes" active="no"/>
+<layer number="21" name="tPlace" color="7" fill="1" visible="yes" active="no"/>
+<layer number="22" name="bPlace" color="7" fill="1" visible="yes" active="no"/>
+<layer number="23" name="tOrigins" color="15" fill="1" visible="yes" active="no"/>
+<layer number="24" name="bOrigins" color="15" fill="1" visible="yes" active="no"/>
+<layer number="25" name="tNames" color="7" fill="1" visible="yes" active="no"/>
+<layer number="26" name="bNames" color="7" fill="1" visible="yes" active="no"/>
+<layer number="27" name="tValues" color="7" fill="1" visible="yes" active="no"/>
+<layer number="28" name="bValues" color="7" fill="1" visible="yes" active="no"/>
 <layer number="29" name="tStop" color="7" fill="3" visible="no" active="no"/>
 <layer number="30" name="bStop" color="7" fill="6" visible="no" active="no"/>
@@
 <layer number="35" name="tGlue" color="7" fill="4" visible="no" active="no"/>
 <layer number="36" name="bGlue" color="7" fill="5" visible="no" active="no"/>
-<layer number="37" name="tTest" color="7" fill="1" visible="no" active="no"/>
-<layer number="38" name="bTest" color="7" fill="1" visible="no" active="no"/>
+<layer number="37" name="tTest" color="7" fill="1" visible="yes" active="no"/>
+<layer number="38" name="bTest" color="7" fill="1" visible="yes" active="no"/>
 <layer number="39" name="tKeepout" color="4" fill="11" visible="no" active="no"/>
 <layer number="40" name="bKeepout" color="1" fill="11" visible="no" active="no"/>
@@
 <layer number="44" name="Drills" color="7" fill="1" visible="no" active="no"/>
 <layer number="45" name="Holes" color="7" fill="1" visible="no" active="no"/>
-<layer number="46" name="Milling" color="3" fill="1" visible="no" active="no"/>
-<layer number="47" name="Measures" color="7" fill="1" visible="no" active="no"/>
-<layer number="48" name="Document" color="7" fill="1" visible="no" active="no"/>
-<layer number="49" name="Reference" color="7" fill="1" visible="no" active="no"/>
-<layer number="50" name="dxf" color="7" fill="1" visible="no" active="no"/>
-<layer number="51" name="tDocu" color="7" fill="1" visible="no" active="no"/>
-<layer number="52" name="bDocu" color="7" fill="1" visible="no" active="no"/>
-<layer number="53" name="tGND_GNDA" color="7" fill="9" visible="no" active="no"/>
-<layer number="54" name="bGND_GNDA" color="1" fill="9" visible="no" active="no"/>
-<layer number="56" name="wert" color="7" fill="1" visible="no" active="no"/>
-<layer number="57" name="tCAD" color="7" fill="1" visible="no" active="no"/>
-<layer number="59" name="tCarbon" color="7" fill="1" visible="no" active="no"/>
-<layer number="60" name="bCarbon" color="7" fill="1" visible="no" active="no"/>
+<layer number="46" name="Milling" color="3" fill="1" visible="yes" active="no"/>
+<layer number="47" name="Measures" color="7" fill="1" visible="yes" active="no"/>
+<layer number="48" name="Document" color="7" fill="1" visible="yes" active="no"/>
+<layer number="49" name="Reference" color="7" fill="1" visible="yes" active="no"/>
+<layer number="50" name="dxf" color="7" fill="1" visible="yes" active="no"/>
+<layer number="51" name="tDocu" color="7" fill="1" visible="yes" active="no"/>
+<layer number="52" name="bDocu" color="7" fill="1" visible="yes" active="no"/>
+<layer number="53" name="tGND_GNDA" color="7" fill="9" visible="yes" active="no"/>
+<layer number="54" name="bGND_GNDA" color="1" fill="9" visible="yes" active="no"/>
+<layer number="56" name="wert" color="7" fill="1" visible="yes" active="no"/>
+<layer number="57" name="tCAD" color="7" fill="1" visible="yes" active="no"/>
+<layer number="59" name="tCarbon" color="7" fill="1" visible="yes" active="no"/>
+<layer number="60" name="bCarbon" color="7" fill="1" visible="yes" active="no"/>
 <layer number="90" name="Modules" color="5" fill="1" visible="yes" active="yes"/>
 <layer number="91" name="Nets" color="2" fill="1" visible="yes" active="yes"/>
@@
 <parts>
 <part name="Q7" library="808_lt" deviceset="2N3904" device=""/>
-<part name="C2" library="rcl" deviceset="C-US" device="050-025X075" value="47p"/>
+<part name="C2" library="rcl" deviceset="C-US" device="025-030X050" value="47p"/>
 <part name="R2" library="rcl" deviceset="R-US_" device="0207/7" value="470k"/>
 <part name="R3" library="rcl" deviceset="R-US_" device="0207/7" value="47k"/>

Commit message: 96pct auto
Parts:
- C3: device rcl:CPOL-USB45181A -> rcl:CPOL-USB45181B
Changed lines of the file:
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@@
 <part name="R3" library="rcl" deviceset="R-US_" device="0207/7" value="47k"/>
 <part name="R4" library="rcl" deviceset="R-US_" device="0207/7" value="220R"/>
-<part name="C3" library="rcl" deviceset="CPOL-US" device="B45181A" value="1uF"/>
+<part name="C3" library="rcl" deviceset="CPOL-US" device="B45181B" value="1uF"/>
 <part name="JCK1" library="erthenvar" deviceset="AUDIO-JACK" device=""/>
 <part name="R1" library="rcl" deviceset="R-US_" device="0207/7" value="100k"/>

Commit message: routed
Parts:
- L6: device rcl:L-US0204/7 -> rcl:L-US0204/5
Changed lines of the file:
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@@
 <part name="C342" library="rcl" deviceset="C-US" device="050-025X075" value="18n"/>
 <part name="P+1" library="supply1" deviceset="+12V" device=""/>
-<part name="L6" library="rcl" deviceset="L-US" device="0204/7" value="45mH"/>
+<part name="L6" library="rcl" deviceset="L-US" device="0204/5" value="45mH"/>
 <part name="C541" library="rcl" deviceset="C-US" device="050-025X075" value="15n"/>
 <part name="GND4" library="supply1" deviceset="GND" device=""/>
