File: eagle/CR78-MB.brd (EAGLE design)
At the start: 100.6 x 80.6 mm, 45 parts, among them Q508 2N3904, Q518 2N3904, Q519 2N3904, Q520 2N3904, Q521 2N3904, Q7 2N3904

Commit message: half schemo
Parts:
- removed 671, R543: 82k, rcl:0207/7
- removed C4, C5: 68n, rcl:C050-025X075
- removed C507: 100/10, rcl:B45181A
- removed D519, D520, D527: (no value), SparkFun-DiscreteSemi:DIODE-1N4148
- removed GU: (no value), con-molex:22-23-2061
- removed Q519, Q520, Q521: 2N3904, 808_lt:TO92
- removed R544, R545: 56k, rcl:0207/7
- removed R546: 2M2, rcl:0207/7
- removed R549, R670, R675: 10k, rcl:0207/7
- removed R550: 820, rcl:0207/7
- removed R672: 47k, rcl:0207/7
- removed R673: 5k6, rcl:0207/7
- removed R674: 15k, rcl:0207/7
- removed R676: 3k9, rcl:0207/7
- removed R677: 18k, rcl:0207/7
- removed VR59: 100K, TR808clone:B64Y
- added C540: 22n, rcl:C050-025X075
- added D524: (no value), SparkFun-DiscreteSemi:DIODE-1N4148
- added IC1: 40106N, 40xx:DIL14
- added MB: 22-23-2051, con-molex:22-23-2051
- added Q1: 2N3904, 808_lt:TO92
- added R566: 470k, rcl:0207/7
- added R567: 820k, rcl:0207/7
- added R568: 10k, rcl:0207/7
- added R569: 4M7, rcl:0207/7
- C342: value 15n -> 18n
- C541: value 22n -> 15n
- R548: value 470k -> 270k
- R570: value 47k -> 100k
- R668: value 56k -> 10k
- moved R668 81.6 mm to (-2.54, -17.8), turned to 0 degrees
- renumbered C531 to C541, C532 to C342, Q508 to Q510, R547 to R570
Connections:
- removed net N$10: R673.1, R674.1, R675.1, R676.2
- removed net N$11: GU.2, R668.1
- removed net N$14: R545.1, VR59.A
- removed net N$22: R543.1, R544.1, R545.2, R672.2
- removed net N$23: D527.C, R672.1
- removed net N$46: D527.A, Q519.1, R670.2
- removed net N$47: Q519.2, R668.2
- removed net N$5: D520.C, Q521.1, R546.2, R675.2
- removed net N$6: C5.2, D520.A, R674.2
- removed net N$8: C4.2, Q521.2, R544.2
- removed net N$9: C4.1, Q520.1, R673.2
- new net +5V: MB.2
- new net VDD: IC1.14
- new net VSS: IC1.7
- net +12V: now also MB.3, R567.2, R568.2, R668.2; no longer GU.4, R549.1, R670.1, R676.1, VR59.E, VR59.S
- net GND: now also C540.2, MB.4, Q1.3, Q510.3, R548.1; no longer C507.-, GU.5, Q519.3, R550.2, R677.1
- net N$1: now also D524.A, Q1.1, R568.1; no longer 671.2, D519.C, R677.2
- net N$12: now also R569.2; no longer R546.1
- net N$2: now also Q1.2, R566.1, R567.1; no longer C5.1, D519.A, Q520.2, R543.2
- net N$20: now also R566.2; no longer 671.1
- net N$24: now also MB.1; no longer GU.1
- net N$27: now also R668.1
- net N$3: no longer GU.3
- net N$4: now also C540.1, D524.C, R569.1; no longer C507.+, Q510.3, Q520.3, Q521.3, R548.1, R549.2, R550.1
- net N$7: now also MB.5; no longer GU.6
Routing:
- net +12V: track 192.6 -> 125.3 mm
- net N$4: track 67.2 -> 0.00 mm
- net GND: track 127.6 -> 97.6 mm
- net N$8: track 28.3 -> 0.00 mm
- net N$7: track 63.7 -> 44.6 mm
- net N$1: track 15.0 -> 0.00 mm
- net N$46: track 14.0 -> 0.00 mm
- net N$10: track 13.2 -> 0.00 mm
- net N$2: track 12.7 -> 0.00 mm
- net N$22: track 11.4 -> 0.00 mm
- net N$5: track 10.6 -> 0.00 mm
- net N$9: track 8.89 -> 0.00 mm
- net N$12: track 14.7 -> 6.12 mm
- net N$6: track 8.22 -> 0.00 mm
- net N$11: track 5.62 -> 0.00 mm
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
Commit message: schemo
Parts:
- removed VR63: 50KB, TR808clone:B64Y
- added C4: 1n5, rcl:C050-025X075
- added C5: 1n8, rcl:C050-025X075
- added C6: 2n2, rcl:C050-025X075
- added R10, R5, R9: 4k7, rcl:0207/7
- added R11, R12, R7: 470k, rcl:0207/7
- added R13, R6, R8: 39k, rcl:0207/7
- added R14: 10k, rcl:0207/7
- added VR1, VR2, VR3: 20K, TR808clone:B64Y
Connections:
- removed net VDD: IC1.14
- removed net VSS: IC1.7
- new net N$10: IC1.10, IC1.13, R13.1
- new net N$11: C5.2, IC1.8, R11.2
- new net N$14: C6.2, IC1.12, R12.2
- new net N$22: C4.2, IC1.4, R7.2
- new net N$23: R6.2, VR1.E
- new net N$25: R8.2, VR2.E
- new net N$26: R13.2, VR3.E
- new net N$28: C4.1, R5.2, VR1.S
- new net N$29: C5.1, R9.2, VR2.S
- new net N$30: C6.1, R10.2, VR3.S
- new net N$5: IC1.2, IC1.3, R6.1
- new net N$6: IC1.6, IC1.9, R8.1
- new net N$8: IC1.5, R9.1
- new net N$9: IC1.11, R10.1
- net +12V: no longer VR63.A
- net +5V: now also IC1.14
- net GND: now also IC1.7, R14.2
- net N$17: now also IC1.1, R5.1; no longer C541.2, VR63.S
- net N$3: now also C541.2, R11.1, R12.1, R14.1, R7.1; no longer VR63.E
Routing:
- net N$17: track 48.8 -> 0.00 mm
- net +12V: track 125.3 -> 85.0 mm
- net N$3: track 20.0 -> 0.00 mm

Commit message: starting brd
Parts:
- removed D524: (no value), SparkFun-DiscreteSemi:DIODE-1N4148
- removed L4: 45mH, rcl:0204/7
- removed Q1: 2N3904, 808_lt:TO92
- added D571: (no value), SparkFun-DiscreteSemi:DIODE-1N4148
- added L6: 45mH, rcl:0204/7
- added Q526: 2N3904, 808_lt:TO92
- moved R14 201.5 mm to (-58.4, 59.7)
- moved C6 189.2 mm to (27.9, 48.3), turned to 180 degrees
- moved R13 174.4 mm to (27.9, 55.9)
- moved VR3 170.8 mm to (29.2, 52.1), turned to 180 degrees
- moved C5 166.7 mm to (25.4, 33.0), turned to 180 degrees
- moved C4 164.2 mm to (7.62, 43.2)
- moved R10 150.2 mm to (27.9, 45.7)
- moved R12 139.3 mm to (10.2, 29.2)
- moved R11 136.8 mm to (10.2, 31.8)
- moved R8 135.9 mm to (27.9, 40.6)
- moved R9 135.0 mm to (7.62, 40.6), turned to 180 degrees
- moved R6 128.4 mm to (7.62, 50.8), turned to 180 degrees
- moved R566 127.7 mm to (35.6, 63.5), turned to 90 degrees
- moved R5 125.9 mm to (7.62, 53.3), turned to 180 degrees
- moved VR2 125.1 mm to (29.2, 36.8), turned to 180 degrees
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Connections:
- net +12V: now also L6.1; no longer L4.1
- net GND: now also Q526.3; no longer Q1.3
- net N$1: now also D571.A, Q526.1; no longer D524.A, Q1.1
- net N$2: now also Q526.2; no longer Q1.2
- net N$27: now also L6.2; no longer L4.2
- net N$4: now also D571.C; no longer D524.C
Routing:
- net GND: track 97.6 -> 0.00 mm, vias 2 -> 0
- net +12V: track 85.0 -> 0.00 mm
- net N$7: track 44.6 -> 0.00 mm
- net N$18: track 24.1 -> 0.00 mm
- net N$16: track 23.1 -> 0.00 mm
- net N$19: track 17.5 -> 0.00 mm
- net N$27: track 12.6 -> 0.00 mm
- net N$13: track 9.09 -> 0.00 mm
- net N$12: track 6.12 -> 0.00 mm
- net N$21: track 4.49 -> 0.00 mm
- net N$15: track 2.84 -> 0.00 mm
- net N$20: track 2.17 -> 0.00 mm
Other:
- board size 100.6 x 80.6 mm -> 100 x 80 mm

Commit message: parts on the brd
Parts:
- C2: device rcl:C050-025X075 -> rcl:C025-030X050
- moved L6 112.6 mm to (44.5, 24.1), turned to 90 degrees
- moved R569 102.9 mm to (43.2, 48.3)
- moved Q510 97.4 mm to (45.7, 31.8)
- moved R568 93.6 mm to (44.5, 52.1), turned to 180 degrees
- moved R3 91.6 mm to (36.8, 22.9)
- moved R4 87.3 mm to (20.3, 17.8), turned to 270 degrees
- moved R668 83.5 mm to (36.8, 33.0), turned to 180 degrees
- moved C541 82.6 mm to (39.4, 40.6), turned to 180 degrees
- moved R14 77.3 mm to (10.2, 24.1)
- moved R2 71.9 mm to (26.7, 24.1), turned to 270 degrees
- moved C2 71.3 mm to (30.5, 24.1), turned to 270 degrees
- moved C540 70.8 mm to (35.6, 49.5), turned to 90 degrees
- moved R570 70.5 mm to (47.0, 41.9), turned to 270 degrees
- moved C1 68.7 mm to (36.8, 25.4), turned to 180 degrees
- moved D571 66.3 mm to (45.7, 55.9)
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
Commit message: 96pct auto
Parts:
- C3: device rcl:B45181A -> rcl:B45181B
- moved R14 36.7 mm to (45.7, 15.2), turned to 180 degrees
- moved R12 36.1 mm to (45.7, 22.9), turned to 90 degrees
- moved R3 30.3 mm to (62.2, 6.35)
- moved R7 30.1 mm to (36.8, 20.3), turned to 180 degrees
- moved C2 29.6 mm to (55.9, 8.89)
- moved Q7 29.6 mm to (47.0, 8.89)
- moved C1 29.6 mm to (62.2, 10.2)
- moved R2 29.0 mm to (52.1, 10.2)
- moved C342 28.5 mm to (61.0, 14.0)
- moved R11 28.1 mm to (36.8, 22.9), turned to 180 degrees
- moved R668 26.4 mm to (58.4, 17.8)
- moved L6 26.2 mm to (68.6, 14.0)
- moved R548 26.2 mm to (64.8, 26.7)
- moved VR2 25.7 mm to (50.8, 22.9), turned to 270 degrees
- moved R1 25.6 mm to (39.4, 11.4), turned to 180 degrees
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Routing:
- net GND: track 0.00 -> 180.0 mm
- net +12V: track 0.00 -> 154.9 mm
- net N$29: track 0.00 -> 46.0 mm
- net N$27: track 0.00 -> 36.1 mm
- net N$3: track 0.00 -> 27.3 mm
- net N$16: track 0.00 -> 22.9 mm
- net N$18: track 0.00 -> 22.1 mm
- net N$22: track 0.00 -> 20.4 mm
- net N$6: track 0.00 -> 19.7 mm
- net N$10: track 0.00 -> 17.3 mm
- net N$14: track 0.00 -> 16.7 mm
- net N$28: track 0.00 -> 16.5 mm
- net N$11: track 0.00 -> 16.1 mm
- net +5V: track 0.00 -> 12.0 mm
- net N$13: track 0.00 -> 11.4 mm
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
Commit message: routed
Parts:
- L6: device rcl:0204/7 -> rcl:0204/5
- moved R668 5.57 mm to (60.7, 12.7)
- moved R13 4.79 mm to (45.7, 49.8)
- moved L6 4.49 mm to (65.5, 17.3), turned to 180 degrees
- moved C342 4.13 mm to (61.7, 9.91)
- moved C1 3.57 mm to (62.0, 6.60)
- moved R3 3.06 mm to (62.0, 3.30)
- moved C3 1.63 mm to (38.1, 4.83)
- moved Q526 1.52 mm to (57.1, 44.2)
- moved Q510 1.37 mm to (62.7, 22.9)
- moved VR3 1.30 mm to (49.8, 43.2), turned to 270 degrees
- moved R548 1.30 mm to (63.5, 26.9)
- moved R568 1.27 mm to (64.8, 41.9)
- moved R11 1.27 mm to (38.1, 22.9)
- moved R566 1.27 mm to (55.9, 52.1)
- moved R567 1.27 mm to (62.2, 50.8)
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Routing:
- net N$7: track 0.00 -> 46.2 mm
- net N$27: track 36.1 -> 17.5 mm
- net GND: track 180.0 -> 196.9 mm
- net N$19: track 0.00 -> 16.8 mm
- net N$10: track 17.3 -> 22.6 mm
- net N$3: track 27.3 -> 22.9 mm
- net N$16: track 22.9 -> 25.5 mm
- net N$20: track 10.2 -> 7.62 mm
- net N$13: track 11.4 -> 9.42 mm
- net N$11: track 16.1 -> 14.4 mm
- net N$24: track 5.08 -> 4.02 mm
- net N$30: track 7.59 -> 8.57 mm
- net N$1: track 7.62 -> 6.64 mm
- net N$23: track 8.89 -> 7.94 mm
- net N$18: track 22.1 -> 21.2 mm
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
Commit message: cutout
Parts:
- moved R669 3.59 mm to (62.7, 51.1)
- moved R567 2.34 mm to (62.7, 48.5)
Routing:
- net N$20: track 7.62 -> 9.76 mm
- net N$2: track 7.41 -> 5.70 mm
- net +12V: track 154.4 -> 153.2 mm
Other:
- board size 100 x 80 mm -> 100 x 80.8 mm
Changed lines of the file:
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@@
 <layer number="44" name="Drills" color="7" fill="1" visible="no" active="yes"/>
 <layer number="45" name="Holes" color="7" fill="1" visible="no" active="yes"/>
-<layer number="46" name="Milling" color="3" fill="1" visible="no" active="yes"/>
+<layer number="46" name="Milling" color="3" fill="1" visible="yes" active="yes"/>
 <layer number="47" name="Measures" color="7" fill="1" visible="no" active="yes"/>
 <layer number="48" name="Document" color="7" fill="1" visible="yes" active="yes"/>
@@
 <wire x1="100" y1="80" x2="0" y2="80" width="0" layer="20"/>
 <wire x1="0" y1="80" x2="0" y2="0" width="0" layer="20"/>
+<wire x1="71.12" y1="1.27" x2="71.12" y2="58.42" width="1.6764" layer="46"/>
+<wire x1="71.12" y1="58.42" x2="69.85" y2="59.69" width="1.6764" layer="46"/>
+<wire x1="69.85" y1="59.69" x2="19.05" y2="59.69" width="1.6764" layer="46"/>
+<wire x1="19.05" y1="59.69" x2="17.78" y2="58.42" width="1.6764" layer="46"/>
+<wire x1="17.78" y1="58.42" x2="17.78" y2="0.762" width="1.6764" layer="46"/>
+<wire x1="17.78" y1="0.762" x2="19.304" y2="-0.762" width="1.6764" layer="46"/>
+<wire x1="19.304" y1="-0.762" x2="69.088" y2="-0.762" width="1.6764" layer="46"/>
+<wire x1="69.088" y1="-0.762" x2="71.12" y2="1.27" width="1.6764" layer="46"/>
+<wire x1="21.082" y1="56.134" x2="22.352" y2="56.134" width="1.6764" layer="46"/>
+<wire x1="22.352" y1="56.134" x2="22.352" y2="54.864" width="1.6764" layer="46"/>
+<wire x1="22.352" y1="54.864" x2="21.082" y2="54.864" width="1.6764" layer="46"/>
+<wire x1="21.082" y1="54.864" x2="21.082" y2="56.134" width="1.6764" layer="46"/>
+<wire x1="21.844" y1="7.874" x2="23.114" y2="7.874" width="1.6764" layer="46"/>
+<wire x1="23.114" y1="7.874" x2="23.114" y2="6.604" width="1.6764" layer="46"/>
+<wire x1="23.114" y1="6.604" x2="21.844" y2="6.604" width="1.6764" layer="46"/>
+<wire x1="21.844" y1="6.604" x2="21.844" y2="7.874" width="1.6764" layer="46"/>
+<wire x1="64.008" y1="56.642" x2="65.278" y2="56.642" width="1.6764" layer="46"/>
+<wire x1="65.278" y1="56.642" x2="65.278" y2="55.372" width="1.6764" layer="46"/>
+<wire x1="65.278" y1="55.372" x2="64.008" y2="55.372" width="1.6764" layer="46"/>
+<wire x1="64.008" y1="55.372" x2="64.008" y2="56.642" width="1.6764" layer="46"/>
 </plain>
 <attributes>
@@
 <element name="R548" library="rcl" package="0207/7" value="270k" x="63.5" y="26.924"/>
 <element name="R566" library="rcl" package="0207/7" value="470k" x="55.88" y="52.07" rot="R90"/>
-<element name="R567" library="rcl" package="0207/7" value="820k" x="62.23" y="50.8"/>
+<element name="R567" library="rcl" package="0207/7" value="820k" x="62.738" y="48.514"/>
 <element name="R568" library="rcl" package="0207/7" value="10k" x="64.77" y="41.91" rot="R270"/>
 <element name="R569" library="rcl" package="0207/7" value="4M7" x="60.96" y="34.29"/>
@@
 <element name="R667" library="rcl" package="0207/7" value="56k" x="44.45" y="53.34"/>
 <element name="R668" library="rcl" package="0207/7" value="10k" x="60.706" y="12.7" rot="R180"/>
-<element name="R669" library="rcl" package="0207/7" value="10k" x="62.23" y="54.61" rot="R180"/>
+<element name="R669" library="rcl" package="0207/7" value="10k" x="62.738" y="51.054" rot="R180"/>
 <element name="R7" library="rcl" package="0207/7" value="470k" x="38.1" y="20.32" rot="R180"/>
 <element name="R8" library="rcl" package="0207/7" value="39k" x="48.26" y="31.75"/>
@@
 <wire x1="56.896" y1="12.7" x2="59.182" y2="9.906" width="0.8128" layer="16"/>
 <wire x1="66.8655" y1="39.6875" x2="64.77" y2="38.1" width="0.8128" layer="16"/>
-<wire x1="66.8655" y1="50.4825" x2="66.8655" y2="39.6875" width="0.8128" layer="16"/>
-<wire x1="66.04" y1="50.8" x2="66.8655" y2="50.4825" width="0.8128" layer="16"/>
-<wire x1="66.04" y1="50.8" x2="66.04" y2="54.61" width="0.8128" layer="16"/>
+<wire x1="66.8655" y1="47.6885" x2="66.8655" y2="39.6875" width="0.8128" layer="16"/>
+<wire x1="66.548" y1="48.514" x2="66.8655" y2="47.6885" width="0.8128" layer="16"/>
+<wire x1="66.548" y1="48.514" x2="66.548" y2="51.054" width="0.8128" layer="16"/>
 <wire x1="31.877" y1="51.943" x2="31.75" y2="52.07" width="0.8128" layer="16"/>
 <wire x1="32.385" y1="53.34" x2="31.877" y2="51.943" width="0.8128" layer="16"/>
 <wire x1="33.7185" y1="57.2135" x2="32.385" y2="53.34" width="0.8128" layer="16"/>
-<wire x1="62.23" y1="57.4675" x2="46.0375" y2="57.4675" width="0.8128" layer="16"/>
+<wire x1="57.404" y1="57.4675" x2="46.0375" y2="57.4675" width="0.8128" layer="16"/>
 <wire x1="46.0375" y1="57.4675" x2="33.7185" y2="57.2135" width="0.8128" layer="16"/>
-<wire x1="66.04" y1="54.61" x2="62.23" y2="57.4675" width="0.8128" layer="16"/>
+<wire x1="66.548" y1="51.054" x2="61.976" y2="51.054" width="0.8128" layer="16"/>
+<wire x1="61.976" y1="51.054" x2="60.96" y2="52.07" width="0.8128" layer="16"/>
+<wire x1="60.96" y1="52.07" x2="57.404" y2="57.4675" width="0.8128" layer="16"/>
 <wire x1="69.1515" y1="32.639" x2="69.1515" y2="25.019" width="0.8128" layer="16"/>
 <wire x1="66.04" y1="37.7825" x2="69.1515" y2="32.639" width="0.8128" layer="16"/>
@@
 <wire x1="55.88" y1="54.61" x2="52.07" y2="54.61" width="0.8128" layer="16"/>
 <wire x1="55.88" y1="55.88" x2="55.88" y2="54.61" width="0.8128" layer="16"/>
-<wire x1="55.88" y1="54.61" x2="58.42" y2="54.61" width="0.8128" layer="16"/>
+<wire x1="55.88" y1="54.61" x2="58.928" y2="51.054" width="0.8128" layer="16"/>
 </signal>
 <signal name="N$21">
@@
 <wire x1="56.134" y1="47.625" x2="57.15" y2="46.101" width="0.8128" layer="16"/>
 <wire x1="55.88" y1="48.26" x2="56.134" y2="47.625" width="0.8128" layer="16"/>
-<wire x1="57.912" y1="48.006" x2="58.42" y2="50.8" width="0.8128" layer="16"/>
+<wire x1="57.912" y1="48.006" x2="58.928" y2="48.514" width="0.8128" layer="16"/>
 <wire x1="57.912" y1="48.006" x2="57.15" y2="46.101" width="0.8128" layer="16"/>
 </signal>

Commit message: moved to corner
Parts:
- moved C2 19.1 mm to (36.8, 8.89)
- moved C342 19.1 mm to (42.7, 9.91)
- moved R566 19.1 mm to (36.8, 52.1)
- moved R569 19.1 mm to (41.9, 34.3)
- moved R667 19.1 mm to (25.4, 53.3)
- moved R668 19.1 mm to (41.7, 12.7)
- moved C3 19.1 mm to (19.1, 4.83)
- moved C4 19.1 mm to (7.87, 33.0)
- moved IC1 19.1 mm to (19.1, 35.6)
- moved JCK1 19.1 mm to (12.7, 0.00)
- moved MB 19.1 mm to (12.7, 52.1)
- moved Q7 19.1 mm to (27.9, 8.89)
- moved R11 19.1 mm to (19.1, 22.9)
- moved R5 19.1 mm to (8.89, 43.2)
- moved R6 19.1 mm to (8.89, 40.6)
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Other:
- board size 100 x 80.8 mm -> 100.8 x 80.8 mm
